File: Circuit Diagram and Schematic/EG-SLDP.kicad_sch (KiCad schematic)
At the start: 12 parts, among them M1 Stepper_Motor_bipolar, M2 Stepper_Motor_bipolar, SW1 SW_Push, SW2 SW_Push, SW3 SW_Push, SW4 SW_Push, U1 TCS3472, U2 CD74HC4067M, U3 2004 LCD

Commit message: Update CAD & Schematic
Parts:
- removed SW1, SW2, SW3, SW4: SW_Push, symbol Switch:SW_Push
- added SW1: Membrane Keypad, symbol Switch:SW_Rotary_1x4_MP
Connections:
- net +12V: now also A3.8 (VIN)
- net +5V: now also A3.5 (+5V)
- net D7: now also A2.13 (~{RESET}); no longer A1.14 (~{SLEEP})
- net D8: now also A1.14 (~{SLEEP}); no longer A2.13 (~{RESET})
- net GND: now also SW1.1
- net SW1: now also SW1.2
- net SW2: now also SW1.3
- net SW3: now also SW1.4
- net SW4: now also SW1.5
- net A0: now reaches A3.9 (A0)
- net A0: now also U2.1 (COM)
- net A1: no longer names the net of A3.10 (A1)
- net A1: no longer U2.1 (COM)
Other:
- note added: "1A - Black 1B - Green 2A - Red 2B - Blue"
- note removed: "1A - Black 1B - Blue 2A - Green 2B - Red"
