File: Schematic/EG-SLDP.kicad_sch (KiCad schematic)
At the start: 9 parts, among them M1 Stepper_Motor_bipolar, M2 Stepper_Motor_bipolar, SW1 Membrane Keypad, U1 TCS3472, U2 CD74HC4067M, U3 2004 LCD

Commit message: add final cad & schematic
Other:
- note added: "1A - Black 1B - Green 2A - Red 2B - Blue Green Black Red Blue"
Changed lines of the file:
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@@
 		)
 	)
-	(text "1A - Black\n1B - Green\n2A - Red\n2B - Blue"
+	(text "1A - Black\n1B - Green\n2A - Red\n2B - Blue\n\nGreen\nBlack\nRed\nBlue"
 		(exclude_from_sim no)
-		(at 70.104 135.89 0)
+		(at 69.85 141.478 0)
 		(effects
 			(font
